File: pcbs/bear/maibadge_bear_v1/maibadge_bear_v1.kicad_sch (KiCad schematic)
At the start: 23 parts, among them J1 Conn_01x04_Socket, SW1 SW_Push, SW2 SW_Push, SW3 SW_Push, SW4 SW_Push, U1 AMS1117-3.3, U10 SK6812SIDE-A-RVS, U12 MS-23C01-G020, U13 FUET-7525-3_6V, U2 ESP32-S3-WROOM-1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

Commit message: minor edits
Connections:
- net GPIO0_BOOT: now also U2.27 (IO0); no longer U2.24 (IO47)
- net buzzer: now also U2.8 (IO15); no longer U2.27 (IO0)
- no-connect marks 0 -> 6
Other:
- moved on the sheet: JP2, U10, U3, U4, U5, U6, U7, U8, U9
