File: pcbs/bear/maibadge_bear_v1/maibadge_bear_v1.kicad_sch (KiCad schematic)
At the start: 19 parts, among them J1 Conn_01x04_Socket, SW1 SW_Push, SW3 SW_Push, SW4 SW_Push, U1 AMS1117-3.3, U10 SK6812SIDE-A-RVS, U13 FUET-7525-3_6V, U2 ESP32-S3-WROOM-1, U3 SK6812SIDE-A-RVS, U4 SK6812SIDE-A-RVS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

Commit message: feat: renaming labels and further touchups
Parts:
- renumbered SW4 to BOOT, SW1 to DEBUG, SW3 to RESET
Changed lines of the file:
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@@
 		(on_board yes)
 		(dnp no)
-		(property "Reference" "SW4"
+		(property "Reference" "BOOT"
 			(at 96.52 132.08 0)
 			(effects
@@
 			(project "maibadge_bear_v1"
 				(path "/8829ea97-d982-42a1-8001-8683a28d2262"
-					(reference "SW4")
+					(reference "BOOT")
 					(unit 1)
 				)
@@
 		(on_board yes)
 		(dnp no)
-		(property "Reference" "SW3"
+		(property "Reference" "RESET"
 			(at 96.52 107.95 0)
 			(effects
@@
 			(project "maibadge_bear_v1"
 				(path "/8829ea97-d982-42a1-8001-8683a28d2262"
-					(reference "SW3")
+					(reference "RESET")
 					(unit 1)
 				)
@@
 		(on_board yes)
 		(dnp no)
-		(property "Reference" "SW1"
+		(property "Reference" "DEBUG"
 			(at 31.75 82.55 0)
 			(effects
@@
 			(project ""
 				(path "/8829ea97-d982-42a1-8001-8683a28d2262"
-					(reference "SW1")
-					(unit 1)
-				)
+					(reference "DEBUG")
+					(unit 1)
+				)

Commit message: feat: labelling components
Parts:
- renumbered BOOT to BOOT1, DEBUG to DEBUG1, GC9A01 to GC9A1, RESET to RESET1
Changed lines of the file:
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@@
 		(on_board yes)
 		(dnp no)
-		(property "Reference" "BOOT"
+		(property "Reference" "BOOT1"
 			(at 96.52 132.08 0)
 			(effects
@@
 			(project "maibadge_bear_v1"
 				(path "/8829ea97-d982-42a1-8001-8683a28d2262"
-					(reference "BOOT")
+					(reference "BOOT1")
 					(unit 1)
 				)
@@
 		(dnp no)
 		(fields_autoplaced yes)
-		(property "Reference" "GC9A01"
+		(property "Reference" "GC9A1"
 			(at -17.615 46.99 0)
 			(effects
@@
 			(project ""
 				(path "/8829ea97-d982-42a1-8001-8683a28d2262"
-					(reference "GC9A01")
+					(reference "GC9A1")
 					(unit 1)
 				)
@@
 		(on_board yes)
 		(dnp no)
-		(property "Reference" "RESET"
+		(property "Reference" "RESET1"
 			(at 96.52 107.95 0)
 			(effects
@@
 			(project "maibadge_bear_v1"
 				(path "/8829ea97-d982-42a1-8001-8683a28d2262"
-					(reference "RESET")
+					(reference "RESET1")
 					(unit 1)
 				)
@@
 		(on_board yes)
 		(dnp no)
-		(property "Reference" "DEBUG"
+		(property "Reference" "DEBUG1"
 			(at 31.75 82.55 0)
 			(effects
@@
 			(project ""
 				(path "/8829ea97-d982-42a1-8001-8683a28d2262"
-					(reference "DEBUG")
-					(unit 1)
-				)
+					(reference "DEBUG1")
+					(unit 1)
+				)
